Commit message: navigation stack implementation

File: Code/catkin_ws/src/PioneerModel/p3dx_description/urdf/pioneer3dx.xacro (robot description, xacro)
@@ -206,5 +206,5 @@
   <link name="camera_link">
     <collision>
-      <origin xyz="0 0 0" rpy="3.141592654 0 0"/>
+      <origin xyz="0 0 0" rpy="0 0 0"/>
       <geometry>
     <box size="${camera_link} ${camera_link} ${camera_link}"/>
@@ -212,5 +212,5 @@
     </collision>
     <visual>
-      <origin xyz="0 0 0" rpy="3.141592654 0 0"/>
+      <origin xyz="0 0 0" rpy="0 0 0"/>
       <geometry>
     <box size="${camera_link} ${camera_link} ${camera_link}"/>
@@ -220,8 +220,42 @@
     <inertial>
       <mass value="1e-5" />
-      <origin xyz="0 0 0" rpy="3.141592654 0 0"/>
+      <origin xyz="0 0 0" rpy="0 0 0"/>
       <inertia ixx="1e-6" ixy="0" ixz="0" iyy="1e-6" iyz="0" izz="1e-6" />
     </inertial>
   </link>
+  <joint name="camera_optical_joint" type="fixed">
+    <axis xyz="0 0 0" />
+    <origin xyz="${camera_link} 0.0 0.0" rpy="-1.58 0 -1.58"/>
+    <parent link="camera_link"/>
+    <child link="camera_optical_frame"/>
+  </joint>
+  <link name="camera_optical_frame">
+  </link>
 	<xacro:property name="camera_link" value="0.05" /> <!-- Size of square 'camera' box -->
+	<!-- lms100 laser -->
+	<link name="lms100">
+		<inertial>
+			<mass value="1e-5" />
+			<origin xyz="0 0 0" rpy="0 0 0" />
+			<inertia ixx="1e-6" ixy="0" ixz="0" iyy="1e-6" iyz="0" izz="1e-6" />
+		</inertial>
+		<visual>
+			<origin xyz="0 0 0" rpy="0 0 0" />
+			<geometry>
+				<mesh filename="package://p3dx_description/meshes/lms100.dae" />
+			</geometry>
+		</visual>
+		<collision>
+			<origin xyz="0 0 0" rpy="0 0 0" />
+			<geometry>
+				<box size="0.1 0.1 0.1" />
+			</geometry>
+		</collision>
+	</link>
+	<joint name="lms100_joint" type="fixed">
+		<axis xyz="0 1 0" />
+		<origin xyz="0.16 0 0.05" rpy="0 0 0" />
+		<parent link="base_link" />
+		<child link="lms100" />
+	</joint>
 </robot>

Commit message: Minor stuff

File: Code/catkin_ws/src/PioneerModel/p3dx_description/urdf/pioneer3dx.xacro (robot description, xacro)
@@ -225,6 +225,6 @@
   </link>
   <joint name="camera_optical_joint" type="fixed">
-    <axis xyz="0 0 0" />
-    <origin xyz="${camera_link} 0.0 0.0" rpy="-1.58 0 -1.58"/>
+    <!-- <axis xyz="0 0 0" /> -->
+    <origin rpy="-1.571 0 -1.571"/>
     <parent link="camera_link"/>
     <child link="camera_optical_frame"/>
@@ -232,4 +232,12 @@
   <link name="camera_optical_frame">
   </link>
+  <joint name="camera_depth_joint" type="fixed">
+    <!-- <axis xyz="0 0 0" /> -->
+    <origin rpy="-1.571 -1.571 -1.571"/>
+    <parent link="camera_link"/>
+    <child link="camera_depth_frame"/>
+  </joint>
+  <link name="camera_depth_frame">
+  </link>
 	<xacro:property name="camera_link" value="0.05" /> <!-- Size of square 'camera' box -->
 	<!-- lms100 laser -->

Commit message: More fiddling with rviz visualisation

File: Code/catkin_ws/src/PioneerModel/p3dx_description/urdf/pioneer3dx.xacro (robot description, xacro)
@@ -233,6 +233,5 @@
   </link>
   <joint name="camera_depth_joint" type="fixed">
-    <!-- <axis xyz="0 0 0" /> -->
-    <origin rpy="-1.571 -1.571 -1.571"/>
+    <origin rpy="-1.571 1.571 -1.571"/>
     <parent link="camera_link"/>
     <child link="camera_depth_frame"/>

Commit message: adjusted the camera position

File: Code/catkin_ws/src/PioneerModel/p3dx_description/urdf/pioneer3dx.xacro (robot description, xacro)
@@ -200,5 +200,5 @@
   <joint name="camera_joint" type="fixed">
     <axis xyz="0 0 0" />
-    <origin xyz="${camera_link} 0.0 0.0" rpy="0 0 0"/>
+    <origin xyz="${camera_link} 0.0 -0.135" rpy="0 0 0"/>
     <parent link="front_sonar"/>
     <child link="camera_link"/>
@@ -240,29 +240,3 @@
   </link>
 	<xacro:property name="camera_link" value="0.05" /> <!-- Size of square 'camera' box -->
-	<!-- lms100 laser -->
-	<link name="lms100">
-		<inertial>
-			<mass value="1e-5" />
-			<origin xyz="0 0 0" rpy="0 0 0" />
-			<inertia ixx="1e-6" ixy="0" ixz="0" iyy="1e-6" iyz="0" izz="1e-6" />
-		</inertial>
-		<visual>
-			<origin xyz="0 0 0" rpy="0 0 0" />
-			<geometry>
-				<mesh filename="package://p3dx_description/meshes/lms100.dae" />
-			</geometry>
-		</visual>
-		<collision>
-			<origin xyz="0 0 0" rpy="0 0 0" />
-			<geometry>
-				<box size="0.1 0.1 0.1" />
-			</geometry>
-		</collision>
-	</link>
-	<joint name="lms100_joint" type="fixed">
-		<axis xyz="0 1 0" />
-		<origin xyz="0.16 0 0.05" rpy="0 0 0" />
-		<parent link="base_link" />
-		<child link="lms100" />
-	</joint>
 </robot>
